File: PCB_Related/GTI_V5/GTI_V5.kicad_pcb (KiCad board)
At the start: 4 copper layers, 155 x 75 mm, 165 parts, among them IC3 MAX253CSA+, IC4 AMC1306M25QDWVRQ1, IC5 AMC1306M25QDWVRQ1, IC6 AMC1306M25QDWVRQ1, IC7 MAX253CSA+, IC8 MAX253CSA+, IC9 AMC1306M25QDWVRQ1, J1 Screw_Terminal_01x03, J2 Screw_Terminal_01x02, J3 Screw_Terminal_01x02, J4 Conn_01x05_Male, J5 Conn_01x02_Male, J6 Conn_01x02_Male, K1 G5LE-1, K2 G5LE-1, Q1 BUZ11, Q2 2N7002, Q3 BUZ11, Q4 BUZ11, Q5 BUZ11, T1 760390014, T2 760390014, T3 760390014, U1 STM32L475RCTx, U2 UCC21520ADW, U3 AZ1117-5.0, U4 NCP1117-3.3_SOT223, U5 UCC21520ADW, Y1 Crystal_GND24

Commit message: PCB now assembled - with these component values
The hardware deadtime resistors on the UCC21520 are 4.7K for a 47ns deadtime. This can always be increased further in software on the STM32L475
Parts:
- C73: value 10uF -> 4.7uF
- D6: value DIODE -> ES1J
- R15, R35, R41, R6: value 2.2R -> 4.7K
- R30: value 4.7K -> 2.2K
- R33, R44: value 1K -> 4.7K
Changed lines of the file:
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@@
       (sketchpadsonfab false)
       (subtractmaskfromsilk false)
-      (outputformat 1)
+      (outputformat 4)
       (mirror false)
       (drillshape 0)
       (scaleselection 1)
-      (outputdirectory "C:/Users/James/Documents/3_Hobby Projects/Grid_Tie_Inverter_v4/Gerbers_PCB4/")
+      (outputdirectory "C:/Users/James/Documents/3_Hobby Projects/Grid_Tie_Inverter_V5/")
     )
   )
@@
   (net 135 "/VDDA_B")
   (net 136 "unconnected-(U1-Pad55)")
-  (net 137 "Net-(K1-Pad1)")
+  (net 137 "Net-(C27-Pad2)")
   (net 138 "Net-(C28-Pad1)")
   (net 139 "Net-(K2-Pad3)")
@@
       (net 15 "/Line_GND") (pintype "passive"))
     (pad "2" thru_hole circle locked (at 10 0 90) (size 1.381 1.381) (drill 0.85) (layers *.Cu *.Mask)
-      (net 137 "Net-(K1-Pad1)") (pintype "passive"))
+      (net 137 "Net-(C27-Pad2)") (pintype "passive"))
     (model "C901U222MZVDBA7317.stp"
       (offset (xyz 4.999999925 2.499999962 7.309999833))
@@
       (effects (font (size 1 1) (thickness 0.15)))
     )
-    (fp_text value "1K" (at 0 1.43 90) (layer "F.Fab") hide
+    (fp_text value "4.7K" (at 0 1.43 90) (layer "F.Fab") hide
       (effects (font (size 1 1) (thickness 0.15)))
     )
@@
       (effects (font (size 1 1) (thickness 0.15)))
     )
-    (fp_text value "10uF" (at 0 1.68 90) (layer "F.Fab") hide
+    (fp_text value "4.7uF" (at 0 1.68 90) (layer "F.Fab") hide
       (effects (font (size 1 1) (thickness 0.15)))
     )
@@
       (net 140 "Net-(C22-Pad2)") (pinfunction "1") (pintype "passive"))
     (pad "7" thru_hole circle locked (at 5 -6 90) (size 1.905 1.905) (drill 1.27) (layers *.Cu *.Mask)
-      (net 137 "Net-(K1-Pad1)") (pinfunction "2") (pintype "passive"))
+      (net 137 "Net-(C27-Pad2)") (pinfunction "2") (pintype "passive"))
     (pad "9" thru_hole circle locked (at -5 -6 90) (size 1.905 1.905) (drill 1.27) (layers *.Cu *.Mask)
       (net 15 "/Line_GND") (pinfunction "4") (pintype "passive"))
@@
       (effects (font (size 1 1) (thickness 0.15)))
     )
-    (fp_text value "4.7K" (at 0 1.43) (layer "F.Fab") hide
+    (fp_text value "2.2K" (at 0 1.43) (layer "F.Fab") hide
       (effects (font (size 1 1) (thickness 0.15)))
     )
@@
       (effects (font (size 0.5 0.5) (thickness 0.1)))
     )
-    (fp_text value "2.2R" (at 0 1.43) (layer "F.Fab") hide
+    (fp_text value "4.7K" (at 0 1.43) (layer "F.Fab") hide
       (effects (font (size 1 1) (thickness 0.15)))
     )
@@
       (effects (font (size 1 1) (thickness 0.15)))
     )
-    (fp_text value "2.2R" (at 0 1.43) (layer "F.Fab") hide
+    (fp_text value "4.7K" (at 0 1.43) (layer "F.Fab") hide
       (effects (font (size 1 1) (thickness 0.15)))
     )
@@
     (fp_line (start -8.25 19.95) (end -8.25 -2.55) (layer "F.Fab") (width 0.1))
     (pad "1" thru_hole rect (at 0 0) (size 2.5 2.5) (drill 1.3) (layers *.Cu *.Mask)
-      (net 137 "Net-(K1-Pad1)") (pintype "passive"))
+      (net 137 "Net-(C27-Pad2)") (pintype "passive"))
     (pad "2" thru_hole oval (at -6 2) (size 2.5 2.5) (drill 1.3) (layers *.Cu *.Mask)
       (net 93 "/Relay") (pintype "passive"))
@@
       (effects (font (size 1 1) (thickness 0.15)))
     )
-    (fp_text value "2.2R" (at 0 1.43) (layer "F.Fab") hide
+    (fp_text value "4.7K" (at 0 1.43) (layer "F.Fab") hide
       (effects (font (size 1 1) (thickness 0.15)))
     )
@@
       (effects (font (size 1 1) (thickness 0.15)))
     )
-    (fp_text value "1K" (at 0 1.43 90) (layer "F.Fab") hide
+    (fp_text value "4.7K" (at 0 1.43 90) (layer "F.Fab") hide
       (effects (font (size 1 1) (thickness 0.15)))
     )
@@
       (effects (font (size 0.5 0.5) (thickness 0.1)))
     )
-    (fp_text value "2.2R" (at 0 1.43) (layer "F.Fab") hide
+    (fp_text value "4.7K" (at 0 1.43) (layer "F.Fab") hide
       (effects (font (size 1 1) (thickness 0.15)))
     )
@@
     (fp_line (start -1 -0.625) (end -1 0.625) (layer "B.Fab") (width 0.1))
     (pad "1" smd roundrect (at -0.9125 0 270) (size 1.025 1.4) (layers "B.Cu" "B.Paste" "B.Mask") (roundrect_rratio 0.243902439)
-      (net 137 "Net-(K1-Pad1)") (pintype "passive"))
+      (net 137 "Net-(C27-Pad2)") (pintype "passive"))
     (pad "2" smd roundrect (at 0.9125 0 270) (size 1.025 1.4) (layers "B.Cu" "B.Paste" "B.Mask") (roundrect_rratio 0.243902439)
       (net 60 "Net-(R5-Pad2)") (pintype "passive"))
@@
       (effects (font (size 1.27 1.27) (thickness 0.254)) (justify mirror))
     )
-    (fp_text value "DIODE" (at 0 0) (layer "B.SilkS") hide
+    (fp_text value "ES1J" (at 0 0) (layer "B.SilkS") hide
       (effects (font (size 1.27 1.27) (thickness 0.254)) (justify mirror))
     )
